Commit message: feat(inner_simulator): simulate on the Webots physics and decide by simulation-based inference

File: etc/URDFs/bottle/bottle.urdf (robot description, URDF)
Before this commit: robot bottle, 1 links, 0 joints
Links:
- link base_link: mass 0.5 -> 0.183

File: etc/URDFs/shadow/shadow.urdf (robot description, URDF)
Before this commit: robot shadow, 17 links, 16 joints
Links:
- link base_footprint: mass None -> 0.001
- link bpearl: mass None -> 0.001
- link camera_360_1: mass None -> 0.001
- link camera_360_2: mass None -> 0.001
- link helios: mass None -> 0.001
- link imu: mass None -> 0.001
- link wheel_left: geometry collision sphere radius=0.1; visual cylinder length=0.05 radius=0.1
- link wheel_right: geometry collision sphere radius=0.1; visual cylinder length=0.05 radius=0.1
- link zed: mass None -> 0.001
- link zed_ranger: mass None -> 0.001
Joints:
- joint caster_back_pitch_joint: type continuous -> fixed
- joint caster_back_roll_joint: type continuous -> fixed
- joint caster_back_yaw_joint: type continuous -> fixed
- joint caster_front_pitch_joint: type continuous -> fixed
- joint caster_front_roll_joint: type continuous -> fixed
- joint caster_front_yaw_joint: type continuous -> fixed
